File: pcb/keyboard.kicad_pcb (KiCad board)
At the start: 2 copper layers, 70 x 84 mm, 25 parts, among them SW1 SW_Push, SW2 SW_Push, SW3 RotaryEncoder_Switch, SW4 SW_Push, SW5 SW_Push, SW6 SW_Push, SW7 SW_Push, SW8 SW_Push, SW9 SW_Push, U1 MODULE-SEEEDUINO-XIAO-RP2040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

Commit message: finish the pcb
Parts:
- moved REF** 46.1 mm to (227.0, 73.0)
- moved REF** 19.8 mm to (185.5, 113.0)
Changed lines of the file:
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@@
 	(footprint "MountingHole:MountingHole_3.2mm_M3"
 		(layer "F.Cu")
-		(at 185.5 93)
+		(at 227 73)
 		(descr "Mounting Hole 3.2mm, M3, no annular, generated by kicad-footprint-generator mountinghole.py")
 		(tags "mountinghole M3")
@@
 	(footprint "MountingHole:MountingHole_3.2mm_M3"
 		(layer "F.Cu")
-		(at 205.25 112.75)
+		(at 185.5 113)
 		(descr "Mounting Hole 3.2mm, M3, no annular, generated by kicad-footprint-generator mountinghole.py")
 		(tags "mountinghole M3")
